File: Caravel-Breakout-Pico-Rev-0.0.kicad_pcb (KiCad board)
At the start: 2 copper layers, 33.1 x 57.2 mm, 71 parts, among them J1 Conn_01x22_Pin, J2 Conn_01x22_Pin, J3 Conn_01x03_Pin, J4 Conn_01x06_Pin, J5 USB_C_Receptacle_USB2.0_14P, J7 Conn_01x03_Pin, J8 Conn_01x02_Pin, SW1 SW_Push - SKQGADE010, SW2 SW_Push - SKQGADE010, U10 W25Q128JVS, U11 RP2040, U12 W25Q16JVUXIQ, U4 LP5907SNX-1.8, U5 TLV71333PDQNR, U7 TLV71333PDQNR, U8 M.2-CONNECTOR-E, Y2 ASE-xxxMHz, Y3 ASE-xxxMHz

Commit message: updated flash chip and added uc button
Parts:
- removed U10: W25Q128JVS, Package_SO:SOIC-8_5.3x5.3mm_P1.27mm
- added SW3: SW_Push - SKQGADE010, 000My_Custom_Library:SW4-SMD-5.2X5.2X1.5MM, F.Cu at (139.9, 99.4)
- added U6: W25Q16JVUXIQ, 000My_Custom_Library:USON-8_UX_2x3x0p6_WIN, F.Cu at (142.6, 104.8)
- C28: renamed from C23; footprint Capacitor_SMD:C_0603_1608Metric -> Capacitor_SMD:C_0402_1005Metric
- moved J3 21.0 mm to (137.6, 90.6)
- moved R16 9.95 mm to (145.2, 102.5)
- moved R15 9.77 mm to (146.2, 102.5)
- moved R12 9.63 mm to (147.2, 102.5)
- moved C28 8.53 mm to (138.0, 106.3), turned to -90 degrees
- moved C27 6.95 mm to (139.0, 106.3), turned to -90 degrees
- moved C26 5.89 mm to (140.0, 106.3), turned to 90 degrees
- moved R14 3.96 mm to (138.5, 102.9), turned to 0 degrees
- moved R13 2.70 mm to (138.5, 103.9), turned to 0 degrees
- moved R17 1.88 mm to (138.5, 104.9), turned to 0 degrees
- moved C25 0.64 mm to (144.4, 92.2), turned to -90 degrees
- moved C19 0.50 mm to (156.5, 84.5)
- renumbered C2 to C1, C38 to C12, C37 to C13, C34 to C15, C28 to C16, C35 to C17, C14 to C18, C29 to C19, C3 to C2, C30 to C20, C17 to C21, C31 to C22, C32 to C23, C33 to C24, C20 to C25, C21 to C26, C22 to C27, C4 to C3, C5 to C4, C24 to C5, C36 to C6, C25 to C7, C26 to C9, J8 to J5, J5 to J6, R6 to R1, R14 to R10, R15 to R11, R16 to R12, R17 to R13, R18 to R14, R19 to R15, R20 to R16, R21 to R17, R7 to R2, R9 to R3, R10 to R4, R22 to R5, R11 to R6, R12 to R7, R13 to R8, R8 to R9, U4 to U1, U12 to U2, U5 to U3, U11 to U4, U7 to U5, U8 to U7, Y3 to Y1
Connections:
- J2 pad 15: /mprj_io[27] -> /CARAVEL_GP27
- J2 pad 16: /mprj_io[26] -> /CARAVEL_GP26
- J2 pad 17: /mprj_io[25] -> /CARAVEL_GP25
- J2 pad 18: /mprj_io[24] -> /CARAVEL_GP24
- J2 pad 19: /mprj_io[23] -> /CARAVEL_GP23
- J2 pad 20: /mprj_io[22] -> /CARAVEL_GP22
- J2 pad 21: /mprj_io[21] -> /CARAVEL_GP21
- J2 pad 22: /mprj_io[20] -> /CARAVEL_GP20
- J4 pad 3: /~{MEM_WP} -> unconnected-(J4-Pin_3-Pad3)
- J4 pad 4: /~{MEM_HOLD} -> unconnected-(J4-Pin_4-Pad4)
- U4 pad 31: unconnected-(U11-GPIO20-Pad31) -> /CARAVEL_GP27
- U4 pad 32: unconnected-(U11-GPIO21-Pad32) -> /CARAVEL_GP26
- U4 pad 34: unconnected-(U11-GPIO22-Pad34) -> /CARAVEL_GP25
- U4 pad 35: unconnected-(U11-GPIO23-Pad35) -> /CARAVEL_GP24
- U4 pad 36: unconnected-(U11-GPIO24-Pad36) -> /CARAVEL_GP23
- U4 pad 37: unconnected-(U11-GPIO25-Pad37) -> /CARAVEL_GP22
- U4 pad 40: unconnected-(U11-GPIO28/ADC2-Pad40) -> /CARAVEL_GP21
- U4 pad 41: unconnected-(U11-GPIO29/ADC3-Pad41) -> /CARAVEL_GP20
- U7 pad 48: /mprj_io[27] -> /CARAVEL_GP27
- U7 pad 50: /mprj_io[26] -> /CARAVEL_GP26
- U7 pad 52: /mprj_io[25] -> /CARAVEL_GP25
- U7 pad 54: /mprj_io[24] -> /CARAVEL_GP24
- U7 pad 56: /mprj_io[23] -> /CARAVEL_GP23
- U7 pad 58: /mprj_io[22] -> /CARAVEL_GP22
- U7 pad 60: /mprj_io[21] -> /CARAVEL_GP21
- U7 pad 62: /mprj_io[20] -> /CARAVEL_GP20
Routing:
- net /CARAVEL_GP21: track 0.00 -> 63.4 mm, vias 0 -> 1
- net /CARAVEL_GP22: track 0.00 -> 58.9 mm, vias 0 -> 1
- net /CARAVEL_GP20: track 0.00 -> 56.4 mm
- net /CARAVEL_GP23: track 0.00 -> 53.9 mm, vias 0 -> 1
- net /mprj_io[20]: track 51.5 -> 0.00 mm
- net /CARAVEL_GP24: track 0.00 -> 49.0 mm, vias 0 -> 1
- net /mprj_io[21]: track 48.7 -> 0.00 mm
- net /mprj_io[22]: track 45.9 -> 0.00 mm
- net /CARAVEL_GP25: track 0.00 -> 45.3 mm, vias 0 -> 1
- net /CARAVEL_GP26: track 0.00 -> 44.8 mm, vias 0 -> 1
- net /mprj_io[23]: track 43.1 -> 0.00 mm
- net /CARAVEL_GP27: track 0.00 -> 41.2 mm, vias 0 -> 1
- net /RUN: track 18.7 -> 59.8 mm, vias 1 -> 2
- net /mprj_io[24]: track 40.3 -> 0.00 mm
- net /mprj_io[25]: track 37.5 -> 0.00 mm
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Other:
- board text added: "nrst"
- board text added: "pico"
- board text added: "μrun"

Commit message: rev 1.3
Parts:
- added R18: 1K, Resistor_SMD:R_0402_1005Metric, F.Cu at (136.3, 80.8)
- moved J3 1.10 mm to (137.6, 91.7)
Connections:
- J1 pad 14: /mprj_io[12] -> /CARAVEL_GP12
- J1 pad 15: /mprj_io[13] -> /CARAVEL_GP13
- J1 pad 2: /mprj_io[19] -> /CARAVEL_GP19
- J1 pad 3: /mprj_io[18] -> /CARAVEL_GP18
- J1 pad 4: /mprj_io[17] -> /CARAVEL_GP17
- J1 pad 5: /mprj_io[16] -> /CARAVEL_GP16
- J1 pad 6: /mprj_io[15] -> /CARAVEL_GP15
- J1 pad 7: /mprj_io[14] -> /CARAVEL_GP14
- U4 pad 12: unconnected-(U4-GPIO9-Pad12) -> /CARAVEL_GP13
- U4 pad 2: unconnected-(U4-GPIO0-Pad2) -> /CARAVEL_GP19
- U4 pad 3: unconnected-(U4-GPIO1-Pad3) -> /CARAVEL_GP18
- U4 pad 4: unconnected-(U4-GPIO2-Pad4) -> /CARAVEL_GP17
- U4 pad 5: unconnected-(U4-GPIO3-Pad5) -> /CARAVEL_GP16
- U4 pad 6: unconnected-(U4-GPIO4-Pad6) -> /CARAVEL_GP15
- U4 pad 7: unconnected-(U4-GPIO5-Pad7) -> /CARAVEL_GP14
- U4 pad 8: unconnected-(U4-GPIO6-Pad8) -> /CARAVEL_GP12
- U7 pad 64: /mprj_io[19] -> /CARAVEL_GP19
- U7 pad 66: /mprj_io[18] -> /CARAVEL_GP18
- U7 pad 68: /mprj_io[17] -> /CARAVEL_GP17
- U7 pad 70: /mprj_io[16] -> /CARAVEL_GP16
- U7 pad 72: /mprj_io[15] -> /CARAVEL_GP15
- U7 pad 73: /mprj_io[12] -> /CARAVEL_GP12
- U7 pad 74: /mprj_io[14] -> /CARAVEL_GP14
- U7 pad 75: /mprj_io[13] -> /CARAVEL_GP13
Routing:
- net /CARAVEL_GP19: track 0.00 -> 63.3 mm, vias 0 -> 1
- net /CARAVEL_GP18: track 0.00 -> 58.5 mm, vias 0 -> 1
- net /CARAVEL_GP17: track 0.00 -> 54.0 mm, vias 0 -> 1
- net /CARAVEL_GP16: track 0.00 -> 53.9 mm, vias 0 -> 1
- net /CARAVEL_GP13: track 0.00 -> 51.6 mm, vias 0 -> 1
- net /CARAVEL_GP12: track 0.00 -> 51.2 mm, vias 0 -> 1
- net /CARAVEL_GP15: track 0.00 -> 48.7 mm, vias 0 -> 1
- net /CARAVEL_GP14: track 0.00 -> 44.9 mm, vias 0 -> 1
- net /mprj_io[19]: track 40.5 -> 0.00 mm
- net /mprj_io[18]: track 37.7 -> 0.00 mm
- net /mprj_io[17]: track 35.0 -> 0.00 mm
- net /mprj_io[16]: track 32.2 -> 0.00 mm
- net /mprj_io[15]: track 29.5 -> 0.00 mm
- net /mprj_io[14]: track 26.7 -> 0.00 mm
- net /mprj_io[12]: track 17.9 -> 0.00 mm
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- added copper zone on In1.Cu, net GND
- added copper zone on In2.Cu, net GND
Other:
- copper layers 2 -> 4
- board text added: "NC"
- board text removed: "~{HOLD}"
- board text removed: "~{WP}"
