File: Caravel-Breakout-Pico-Rev-0.0.kicad_sch (KiCad schematic)
At the start: 73 parts, among them J1 Conn_01x22_Pin, J2 Conn_01x22_Pin, J3 Conn_01x03_Pin, J4 Conn_01x06_Pin, J5 USB_C_Receptacle_USB2.0_14P, J7 Conn_01x03_Pin, J8 Conn_01x02_Pin, SW1 SW_Push - SKQGADE010, SW2 SW_Push - SKQGADE010, U10 W25Q128JVS, U11 RP2040, U12 W25Q16JVUXIQ, U4 LP5907SNX-1.8, U5 TLV71333PDQNR, U7 TLV71333PDQNR, U8 M.2-CONNECTOR-E, U9 W25Q32FVSS, Y2 ASE-xxxMHz, Y3 ASE-xxxMHz

Commit message: updated flash chip and added uc button
Parts:
- removed U10: W25Q128JVS, Package_SO:SOIC-8_5.3x5.3mm_P1.27mm, symbol Memory_Flash:W25Q128JVS
- added SW3: SW_Push - SKQGADE010, 000My_Custom_Library:SW4-SMD-5.2X5.2X1.5MM, symbol Switch:SW_Push
- added U6: W25Q16JVUXIQ, 000My_Custom_Library:USON-8_UX_2x3x0p6_WIN, symbol Memory_Flash:W25Q128JVS
- added U9: W25Q128JVS, Package_SO:SOIC-8_5.3x5.3mm_P1.27mm, symbol Memory_Flash:W25Q128JVS
- C28: renamed from C23; footprint Capacitor_SMD:C_0603_1608Metric -> Capacitor_SMD:C_0402_1005Metric
- renumbered C2 to C1, C38 to C12, C37 to C13, C27 to C14, C34 to C15, C28 to C16, C35 to C17, C14 to C18, C29 to C19, C3 to C2, C30 to C20, C17 to C21, C31 to C22, C32 to C23, C33 to C24, C20 to C25, C21 to C26, C22 to C27, C4 to C3, C5 to C4, C24 to C5, C36 to C6, C25 to C7, C26 to C9, J8 to J5, J5 to J6, R6 to R1, R14 to R10, R15 to R11, R16 to R12, R17 to R13, R18 to R14, R19 to R15, R20 to R16, R21 to R17, R7 to R2, R9 to R3, R10 to R4, R22 to R5, R11 to R6, R12 to R7, R13 to R8, R8 to R9, U4 to U1, U12 to U2, U5 to U3, U11 to U4, U7 to U5, U8 to U7, U9 to U8, Y3 to Y1
Connections:
- net mprj_io[20] is gone; now on net CARAVEL_GP20: J2.22 (Pin_22), U7.62 (P54)
- net mprj_io[21] is gone; now on net CARAVEL_GP21: J2.21 (Pin_21), U7.60 (P52)
- net mprj_io[22] is gone; now on net CARAVEL_GP22: J2.20 (Pin_20), U7.58 (P50)
- net mprj_io[23] is gone; now on net CARAVEL_GP23: J2.19 (Pin_19), U7.56 (P48)
- net mprj_io[24] is gone; now on net CARAVEL_GP24: J2.18 (Pin_18), U7.54 (P46)
- net mprj_io[25] is gone; now on net CARAVEL_GP25: J2.17 (Pin_17), U7.52 (P44)
- net mprj_io[26] is gone; now on net CARAVEL_GP26: J2.16 (Pin_16), U7.50 (P42)
- net mprj_io[27] is gone; now on net CARAVEL_GP27: J2.15 (Pin_15), U7.48 (P40)
- net +3V3_CARAVEL: now also U6.8 (VCC)
- net Caravel_CSB: now also U6.1 (~{CS})
- net Caravel_D0: now also U6.5 (DI/IO_{0})
- net Caravel_D1: now also U6.2 (DO/IO_{1})
- net Caravel_SCK: now also U6.6 (CLK)
- net GND: now also SW3.2, U6.4 (GND)
- net RUN: now also SW3.1
- net ~{MEM_HOLD}: now also U6.7 (~{HOLD}/~{RESET}/IO_{3}); no longer J4.4 (Pin_4)
- net ~{MEM_WP}: now also U6.3 (~{WP}/IO_{2}); no longer J4.3 (Pin_3)
- net CARAVEL_GP27: now reaches U4.31 (GPIO20)
- net CARAVEL_GP26: now reaches U4.32 (GPIO21)
- net CARAVEL_GP25: now reaches U4.34 (GPIO22)
- net CARAVEL_GP24: now reaches U4.35 (GPIO23)
- net CARAVEL_GP23: now reaches U4.36 (GPIO24)
- net CARAVEL_GP22: now reaches U4.37 (GPIO25)
- net CARAVEL_GP21: now reaches U4.40 (GPIO28/ADC2)
- net CARAVEL_GP20: now reaches U4.41 (GPIO29/ADC3)
- no-connect marks 31 -> 25

Commit message: rev 1.3
Parts:
- added R18: 1K, Resistor_SMD:R_0402_1005Metric, symbol Device:R
Connections:
- net mprj_io[12] is gone; now on net CARAVEL_GP12: J1.14 (Pin_14), U7.73 (P65)
- net mprj_io[13] is gone; now on net CARAVEL_GP13: J1.15 (Pin_15), U7.75 (P67)
- net mprj_io[14] is gone; now on net CARAVEL_GP14: J1.7 (Pin_7), U7.74 (P66)
- net mprj_io[15] is gone; now on net CARAVEL_GP15: J1.6 (Pin_6), U7.72 (P64)
- net mprj_io[16] is gone; now on net CARAVEL_GP16: J1.5 (Pin_5), U7.70 (P62)
- net mprj_io[17] is gone; now on net CARAVEL_GP17: J1.4 (Pin_4), U7.68 (P60)
- net mprj_io[18] is gone; now on net CARAVEL_GP18: J1.3 (Pin_3), U7.66 (P58)
- net mprj_io[19] is gone; now on net CARAVEL_GP19: J1.2 (Pin_2), U7.64 (P56)
- net +3V3_MAIN: now also R18.2
- net CARAVEL_PWR: now also R18.1
- net CARAVEL_GP13: now reaches U4.12 (GPIO9)
- net CARAVEL_GP19: now reaches U4.2 (GPIO0)
- net CARAVEL_GP18: now reaches U4.3 (GPIO1)
- net CARAVEL_GP17: now reaches U4.4 (GPIO2)
- net CARAVEL_GP16: now reaches U4.5 (GPIO3)
- net CARAVEL_GP15: now reaches U4.6 (GPIO4)
- net CARAVEL_GP14: now reaches U4.7 (GPIO5)
- net CARAVEL_GP12: now reaches U4.8 (GPIO6)
- no-connect marks 25 -> 18
Other:
- note added: "Pico Module"
- note added: "Pico SPI interface with HKSPI"
- note removed: "*ACBUS8-9 are not configurable as GPIOs in MPSSE mode"
- note removed: "Consider driving with Pico GPIOs"
- note removed: "FTDI Module"
- note removed: "FTDI SPI interface with HKSPI"
- note removed: "consider replacing with W25Q128JVSIQ"
